File: temperature_controller.kicad_pcb (KiCad board)
At the start: 2 copper layers, 100 x 120 mm, 68 parts, among them P1 Ext. Mod/Monitor, Q1 IRL_450, U1 OP497, U2 OP497, U3 ED2610, U4 R_th, U5 INA188, U6 R_heat, U7 AD780

Commit message: final design
Parts:
- added REF**: Via-0.6mm, footprints:Via-0.6mm, F.Cu at (115.0, 134.2)
- added REF**: Via-0.6mm, footprints:Via-0.6mm, F.Cu at (89.9, 133.5)
- added REF**: Via-0.6mm, footprints:Via-0.6mm, F.Cu at (89.5, 136.7)
- added REF**: Via-0.6mm, footprints:Via-0.6mm, F.Cu at (73.3, 139.3)
- added REF**: Via-0.6mm, footprints:Via-0.6mm, F.Cu at (70.8, 142.0)
- added REF**: Via-0.6mm, footprints:Via-0.6mm, F.Cu at (63.1, 139.4)
- added REF**: Via-0.6mm, footprints:Via-0.6mm, F.Cu at (64.3, 141.0)
- added REF**: Via-0.6mm, footprints:Via-0.6mm, F.Cu at (107.5, 130.8)
- added REF**: Via-0.6mm, footprints:Via-0.6mm, F.Cu at (98.0, 137.3)
- added REF**: Via-0.6mm, footprints:Via-0.6mm, F.Cu at (99.6, 136.4)
- added REF**: Via-0.6mm, footprints:Via-0.6mm, F.Cu at (56.5, 149.9)
- added REF**: Via-0.6mm, footprints:Via-0.6mm, F.Cu at (61.7, 149.7)
- added REF**: Via-0.6mm, footprints:Via-0.6mm, F.Cu at (80.1, 134.6)
- added REF**: Via-0.6mm, footprints:Via-0.6mm, F.Cu at (86.2, 133.0)
- added REF**: Via-0.6mm, footprints:Via-0.6mm, F.Cu at (86.0, 134.2)
Other:
- board text added: "Temperature Controller v1 unipolar output, 0.6A max Shreyas Potnis Vutha Labs"
Changed lines of the file:
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@@
 (kicad_pcb (version 4) (host pcbnew 4.0.2-stable)
   (general
-    (links 133)
+    (links 148)
     (no_connects 0)
-    (area 49.912 48.002 150.075001 192.702001)
+    (area 49.924999 49.924999 150.075001 170.075001)
     (thickness 1.6)
-    (drawings 4)
+    (drawings 5)
     (tracks 378)
     (zones 0)
-    (modules 68)
+    (modules 83)
     (nets 45)
   )
   (page A4)
+  (title_block
+    (title "Temperature Controller")
+    (rev v1)
+    (company "Vutha Labs")
+  )
   (layers
     (0 F.Cu signal)
@@
     (visible_elements 7FFFFFFF)
     (pcbplotparams
-      (layerselection 0x00030_80000001)
+      (layerselection 0x010e0_80000001)
       (usegerberextensions false)
       (excludeedgelayer true)
@@
       (outputformat 1)
       (mirror false)
-      (drillshape 1)
+      (drillshape 0)
       (scaleselection 1)
-      (outputdirectory ""))
+      (outputdirectory gerber))
   )
   (net 0 "")
@@
   )
   (module footprints:Via-0.6mm (layer F.Cu)
+    (at 114.9985 134.1755)
+    (fp_text reference REF** (at 0 1.27) (layer F.SilkS) hide
+      (effects (font (size 0.127 0.127) (thickness 0.03175)))
+    )
+    (fp_text value Via-0.6mm (at 0 -1.27) (layer F.Fab) hide
+      (effects (font (size 0.127 0.127) (thickness 0.03175)))
+    )
+    (pad 1 thru_hole circle (at 0 0) (size 0.6 0.6) (drill 0.3) (layers *.Cu)
+      (net 2 GND) (zone_connect 2))
+  )
+  (module footprints:Via-0.6mm (layer F.Cu)
+    (at 107.5055 130.81)
+    (fp_text reference REF** (at 0 1.27) (layer F.SilkS) hide
+      (effects (font (size 0.127 0.127) (thickness 0.03175)))
+    )
+    (fp_text value Via-0.6mm (at 0 -1.27) (layer F.Fab) hide
+      (effects (font (size 0.127 0.127) (thickness 0.03175)))
+    )
+    (pad 1 thru_hole circle (at 0 0) (size 0.6 0.6) (drill 0.3) (layers *.Cu)
+      (net 2 GND) (zone_connect 2))
+  )
+  (module footprints:Via-0.6mm (layer F.Cu)
+    (at 98.044 137.287)
+    (fp_text reference REF** (at 0 1.27) (layer F.SilkS) hide
+      (effects (font (size 0.127 0.127) (thickness 0.03175)))
+    )
+    (fp_text value Via-0.6mm (at 0 -1.27) (layer F.Fab) hide
+      (effects (font (size 0.127 0.127) (thickness 0.03175)))
+    )
+    (pad 1 thru_hole circle (at 0 0) (size 0.6 0.6) (drill 0.3) (layers *.Cu)
+      (net 2 GND) (zone_connect 2))
+  )
+  (module footprints:Via-0.6mm (layer F.Cu)
+    (at 99.6315 136.398)
+    (fp_text reference REF** (at 0 1.27) (layer F.SilkS) hide
+      (effects (font (size 0.127 0.127) (thickness 0.03175)))
+    )
+    (fp_text value Via-0.6mm (at 0 -1.27) (layer F.Fab) hide
+      (effects (font (size 0.127 0.127) (thickness 0.03175)))
+    )
+    (pad 1 thru_hole circle (at 0 0) (size 0.6 0.6) (drill 0.3) (layers *.Cu)
+      (net 2 GND) (zone_connect 2))
+  )
+  (module footprints:Via-0.6mm (layer F.Cu)
+    (at 56.4515 149.86)
+    (fp_text reference REF** (at 0 1.27) (layer F.SilkS) hide
+      (effects (font (size 0.127 0.127) (thickness 0.03175)))
+    )
+    (fp_text value Via-0.6mm (at 0 -1.27) (layer F.Fab) hide
+      (effects (font (size 0.127 0.127) (thickness 0.03175)))
+    )
+    (pad 1 thru_hole circle (at 0 0) (size 0.6 0.6) (drill 0.3) (layers *.Cu)
+      (net 2 GND) (zone_connect 2))
+  )
+  (module footprints:Via-0.6mm (layer F.Cu)
+    (at 61.722 149.733)
+    (fp_text reference REF** (at 0 1.27) (layer F.SilkS) hide
+      (effects (font (size 0.127 0.127) (thickness 0.03175)))
+    )
+    (fp_text value Via-0.6mm (at 0 -1.27) (layer F.Fab) hide
+      (effects (font (size 0.127 0.127) (thickness 0.03175)))
+    )
+    (pad 1 thru_hole circle (at 0 0) (size 0.6 0.6) (drill 0.3) (layers *.Cu)
+      (net 2 GND) (zone_connect 2))
+  )
+  (module footprints:Via-0.6mm (layer F.Cu)
+    (at 80.137 134.62)
+    (fp_text reference REF** (at 0 1.27) (layer F.SilkS) hide
+      (effects (font (size 0.127 0.127) (thickness 0.03175)))
+    )
+    (fp_text value Via-0.6mm (at 0 -1.27) (layer F.Fab) hide
+      (effects (font (size 0.127 0.127) (thickness 0.03175)))
+    )
+    (pad 1 thru_hole circle (at 0 0) (size 0.6 0.6) (drill 0.3) (layers *.Cu)
+      (net 2 GND) (zone_connect 2))
+  )
+  (module footprints:Via-0.6mm (layer F.Cu)
+    (at 86.233 133.0325)
+    (fp_text reference REF** (at 0 1.27) (layer F.SilkS) hide
+      (effects (font (size 0.127 0.127) (thickness 0.03175)))
+    )
+    (fp_text value Via-0.6mm (at 0 -1.27) (layer F.Fab) hide
+      (effects (font (size 0.127 0.127) (thickness 0.03175)))
+    )
+    (pad 1 thru_hole circle (at 0 0) (size 0.6 0.6) (drill 0.3) (layers *.Cu)
+      (net 2 GND) (zone_connect 2))
+  )
+  (module footprints:Via-0.6mm (layer F.Cu)
+    (at 85.979 134.1755)
+    (fp_text reference REF** (at 0 1.27) (layer F.SilkS) hide
+      (effects (font (size 0.127 0.127) (thickness 0.03175)))
+    )
+    (fp_text value Via-0.6mm (at 0 -1.27) (layer F.Fab) hide
+      (effects (font (size 0.127 0.127) (thickness 0.03175)))
+    )
+    (pad 1 thru_hole circle (at 0 0) (size 0.6 0.6) (drill 0.3) (layers *.Cu)
+      (net 2 GND) (zone_connect 2))
+  )
+  (module footprints:Via-0.6mm (layer F.Cu)
+    (at 89.8525 133.477)
+    (fp_text reference REF** (at 0 1.27) (layer F.SilkS) hide
+      (effects (font (size 0.127 0.127) (thickness 0.03175)))
+    )
+    (fp_text value Via-0.6mm (at 0 -1.27) (layer F.Fab) hide
+      (effects (font (size 0.127 0.127) (thickness 0.03175)))
+    )
+    (pad 1 thru_hole circle (at 0 0) (size 0.6 0.6) (drill 0.3) (layers *.Cu)
+      (net 2 GND) (zone_connect 2))
+  )
+  (module footprints:Via-0.6mm (layer F.Cu)
+    (at 89.4715 136.652)
+    (fp_text reference REF** (at 0 1.27) (layer F.SilkS) hide
+      (effects (font (size 0.127 0.127) (thickness 0.03175)))
+    )
+    (fp_text value Via-0.6mm (at 0 -1.27) (layer F.Fab) hide
+      (effects (font (size 0.127 0.127) (thickness 0.03175)))
+    )
+    (pad 1 thru_hole circle (at 0 0) (size 0.6 0.6) (drill 0.3) (layers *.Cu)
+      (net 2 GND) (zone_connect 2))
+  )
+  (module footprints:Via-0.6mm (layer F.Cu)
+    (at 73.279 139.2555)
+    (fp_text reference REF** (at 0 1.27) (layer F.SilkS) hide
+      (effects (font (size 0.127 0.127) (thickness 0.03175)))
+    )
+    (fp_text value Via-0.6mm (at 0 -1.27) (layer F.Fab) hide
+      (effects (font (size 0.127 0.127) (thickness 0.03175)))
+    )
+    (pad 1 thru_hole circle (at 0 0) (size 0.6 0.6) (drill 0.3) (layers *.Cu)
+      (net 2 GND) (zone_connect 2))
+  )
+  (module footprints:Via-0.6mm (layer F.Cu)
+    (at 70.8025 142.0495)
+    (fp_text reference REF** (at 0 1.27) (layer F.SilkS) hide
+      (effects (font (size 0.127 0.127) (thickness 0.03175)))
+    )
+    (fp_text value Via-0.6mm (at 0 -1.27) (layer F.Fab) hide
+      (effects (font (size 0.127 0.127) (thickness 0.03175)))
+    )
+    (pad 1 thru_hole circle (at 0 0) (size 0.6 0.6) (drill 0.3) (layers *.Cu)
+      (net 2 GND) (zone_connect 2))
+  )
+  (module footprints:Via-0.6mm (layer F.Cu)
+    (at 63.119 139.3825)
+    (fp_text reference REF** (at 0 1.27) (layer F.SilkS) hide
+      (effects (font (size 0.127 0.127) (thickness 0.03175)))
+    )
+    (fp_text value Via-0.6mm (at 0 -1.27) (layer F.Fab) hide
+      (effects (font (size 0.127 0.127) (thickness 0.03175)))
+    )
+    (pad 1 thru_hole circle (at 0 0) (size 0.6 0.6) (drill 0.3) (layers *.Cu)
+      (net 2 GND) (zone_connect 2))
+  )
+  (module footprints:Via-0.6mm (layer F.Cu)
+    (at 64.3255 141.0335)
+    (fp_text reference REF** (at 0 1.27) (layer F.SilkS) hide
+      (effects (font (size 0.127 0.127) (thickness 0.03175)))
+    )
+    (fp_text value Via-0.6mm (at 0 -1.27) (layer F.Fab) hide
+      (effects (font (size 0.127 0.127) (thickness 0.03175)))
+    )
+    (pad 1 thru_hole circle (at 0 0) (size 0.6 0.6) (drill 0.3) (layers *.Cu)
+      (net 2 GND) (zone_connect 2))
+  )
+  (module footprints:Via-0.6mm (layer F.Cu)
     (at 139.7635 120.777)
     (fp_text reference REF** (at 0 1.27) (layer F.SilkS) hide
@@
       (net 2 GND) (zone_connect 2))
   )
+  (gr_text "Temperature Controller v1\nunipolar output, 0.6A max\n\nShreyas Potnis\nVutha Labs\n" (at 131.318 60.579) (layer F.SilkS)
+    (effects (font (size 1.5 1.5) (thickness 0.3)))
+  )
   (gr_line (start 50 50) (end 50 170) (angle 90) (layer Edge.Cuts) (width 0.15))
