File: temperature_controller.sch (KiCad schematic (older format))
At the start: 65 parts, among them P1 Ext. Mod/Monitor, Q1 IRL_450, U1 OP497, U2 OP497, U3 ED2610, U4 R_th, U5 INA188, U6 R_heat, U7 AD780

Commit message: final design
Parts:
- R14: value 10k -> 100k
Changed lines of the file:
@@
 LIBS:valves
 LIBS:all_components
+LIBS:temperature_controller-cache
 EELAYER 25 0
 EELAYER END
@@
 P 4200 3600
 F 0 "R14" V 4280 3600 50  0000 C CNN
-F 1 "10k" V 4200 3600 50  0000 C CNN
+F 1 "100k" V 4200 3600 50  0000 C CNN
 F 2 "Resistors_SMD:R_0603_HandSoldering" V 4130 3600 50  0001 C CNN
 F 3 "" H 4200 3600 50  0000 C CNN
